File: hardware/mss/schematics/Arduino Uno Hat/Arduino Uno Hat.kicad_pcb (KiCad board)
At the start: 2 copper layers, 68.6 x 53.3 mm, 17 parts, among them J1 Power, J2 Digital/PWM, J3 Analog, J4 Digital/PWM, J5 LED_STRIP, SW1 SPKR, SW2 RST

Commit message: Updated silkscreen on arduino uno hat
Other:
- board text added: "+"
- board text added: "-"
- board text added: "D"
- board text added: "OV"
Changed lines of the file:
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@@
 		(tags "connector JST XH horizontal")
 		(property "Reference" "J5"
-			(at 2.5 -5.1 90)
+			(at 2.5 -3 90)
 			(layer "F.SilkS")
 			(effects
@@
 		(property "Value" "LED_STRIP"
 			(at 2.5 8.8 90)
-			(layer "F.Fab")
+			(layer "F.SilkS")
 			(effects
 				(font
@@
 		(property "Value" "SPKR"
 			(at 3.81 3.11 0)
-			(layer "F.Fab")
+			(layer "F.SilkS")
 			(effects
 				(font
@@
 		(property "Value" "Speaker"
 			(at 3.81 8.89 90)
-			(layer "F.Fab")
+			(layer "F.SilkS")
 			(effects
 				(font
@@
 		)
 		(property "Value" "LED"
-			(at 1.27 3.96 0)
+			(at 1.27 2.5 0)
 			(layer "F.Fab")
 			(effects
@@
 		(layer "Edge.Cuts")
 	)
+	(gr_text "+"
+		(at 114.5 57.5 0)
+		(layer "F.SilkS")
+		(effects
+			(font
+				(size 1.5 1.5)
+				(thickness 0.15)
+			)
+			(justify left bottom)
+		)
+	)
+	(gr_text "OV"
+		(at 105 78.5 0)
+		(layer "F.SilkS")
+		(effects
+			(font
+				(size 1 1)
+				(thickness 0.15)
+			)
+			(justify left bottom)
+		)
+	)
+	(gr_text "-"
+		(at 115 63.5 0)
+		(layer "F.SilkS")
+		(effects
+			(font
+				(size 1 1)
+				(thickness 0.15)
+			)
+			(justify left bottom)
+		)
+	)
 	(gr_text "https://openquartermaster.com/"
 		(at 120.5 94.5 0)
@@
 			)
 			(justify left bottom)
+		)
+	)
+	(gr_text "D"
+		(at 115 60.5 0)
+		(layer "F.SilkS")
+		(effects
+			(font
+				(size 1 1)
+				(thickness 0.15)
+			)
+			(justify left bottom)
